File: Noiseless Switching Supply.kicad_pcb (KiCad board)
At the start: 2 copper layers, 50 x 31 mm, 50 parts, among them J1 JST S2B-ZR-SMA4-TF, J2 JST S3B-ZR-SMA4-TF, U1 LT8607, U2 LT8607, U3 LT3045, U4 LT3094

Commit message: Add Comments for rev 2
Other:
- board text added: "01000001"
- board text added: "1.0.0"
- board text added: "Silent Split Supply"
- board text removed: "Silent Split Supply Rev 1"
Changed lines of the file:
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@@
   (general
     (thickness 1.6)
-    (drawings 12)
+    (drawings 14)
     (tracks 173)
     (zones 0)
@@
       (outputformat 1)
       (mirror false)
-      (drillshape 1)
+      (drillshape 0)
       (scaleselection 1)
-      (outputdirectory ""))
+      (outputdirectory "Output/"))
   )
   (net 0 "")
@@
     )
   )
-  (gr_text "Silent Split Supply Rev 1" (at 150.25 118) (layer F.SilkS)
+  (gr_text 1.0.0 (at 158.2 119.2) (layer F.SilkS)
     (effects (font (size 1.5 1.5) (thickness 0.3)))
   )
+  (gr_text 01000001 (at 145.2 119.2) (layer F.SilkS)
+    (effects (font (size 1.5 1.5) (thickness 0.3)))
+  )
+  (gr_text "Silent Split Supply" (at 150.25 117) (layer F.SilkS)
+    (effects (font (size 1.5 1.5) (thickness 0.3)))
+  )

Commit message: 2.0.0 Release
Parts:
- removed C11, C12: 22uF, Capacitor_SMD:C_1206_3216Metric
- removed H1, H2, H3, H4: MountingHole_Pad, MountingHole:MountingHole_3.2mm_M3_Pad
- removed U2: LT8607, Package_SO:MSOP-10-1EP_3x3mm_P0.5mm_EP1.68x1.88mm
- added D4: D_Small, Diode_SMD:D_SOD-123, F.Cu at (144.0, 102.5)
- added D5: D_Small, Diode_SMD:D_SOD-123, F.Cu at (143.0, 115.0)
- added L3: 10u, Inductor_SMD:L_Wuerth_MAPI-4030, F.Cu at (143.5, 110.0)
- added PCB1: Board_Module, PCB:PCB_Board_50x31, F.Cu at (149.0, 105.0)
- added R18: 18k, Resistor_SMD:R_0402_1005Metric, F.Cu at (153.5, 112.0)
- added R19: 750k, Resistor_SMD:R_0402_1005Metric, F.Cu at (152.5, 112.0)
- added R20: 0R, Resistor_SMD:R_0402_1005Metric, F.Cu at (165.5, 99.0)
- added R21: 0R, Resistor_SMD:R_0402_1005Metric, F.Cu at (165.5, 111.0)
- C1, C2: value 4.7uF -> 1uF; footprint Capacitor_SMD:C_1206_3216Metric -> Capacitor_SMD:C_0402_1005Metric
- C10, C9: value 100nF -> 10p
- C13, C14: value 4.7uF -> 10u
- C15, C16: value 470nF -> 1u; footprint Capacitor_SMD:C_0402_1005Metric -> Capacitor_SMD:C_1206_3216Metric
- C3: value 1uF -> 2.2uF
- C4: value 1uF -> 100n
- C5: value 10nF -> 2.2uF
- C6: value 10nF -> 100n
- C7, C8: value 100nF -> 10u; footprint Capacitor_SMD:C_0402_1005Metric -> Capacitor_SMD:C_1206_3216Metric
- L1, L2: value L -> 10u; footprint Inductor_SMD:L_Wuerth_MAPI-4020 -> Inductor_SMD:L_Wuerth_MAPI-4030
- R10: value R_Small -> 750k
- R11, R8: value R_Small -> 18k
- R2: value 0R -> 82k
- R3: value 0R -> 100k
- R4, R5: value DNP -> 100k
- R6: value 40.2k -> 390k
- R7: value 40.2k -> 18k
- R9: value R_Small -> 390k
- U1: value LT8607 -> LT8471; footprint Package_SO:MSOP-10-1EP_3x3mm_P0.5mm_EP1.68x1.88mm -> Package_DFN_QFN:QFN-28-1EP_4x5mm_P0.5mm_EP2.65x3.65mm
- moved R10 23.8 mm to (160.5, 104.0), turned to 180 degrees
- moved R11 20.2 mm to (158.5, 104.0), turned to 180 degrees
- moved R8 17.1 mm to (139.0, 112.0), turned to 270 degrees
- moved R7 14.5 mm to (137.5, 97.5), turned to 270 degrees
- moved C4 14.2 mm to (136.5, 100.0), turned to 90 degrees
- moved L1 13.6 mm to (136.5, 110.0), turned to 0 degrees
- moved L2 11.5 mm to (147.5, 102.5), turned to 180 degrees
- moved R3 11.4 mm to (138.5, 100.0), turned to 90 degrees
- moved R2 11.2 mm to (137.5, 100.0), turned to 90 degrees
- moved C5 10.3 mm to (143.5, 106.0), turned to 270 degrees
- moved C14 10.1 mm to (148.0, 115.0), turned to 270 degrees
- moved C13 10.0 mm to (143.5, 96.5), turned to 180 degrees
- moved R6 10.00 mm to (137.5, 95.5), turned to 270 degrees
- moved C3 9.06 mm to (148.5, 106.0), turned to 270 degrees
- moved U1 8.28 mm to (139.5, 105.0), turned to 270 degrees
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Connections:
- C10 pad 1: GND -> Net-(C10-Pad1)
- C10 pad 2: Net-(C10-Pad2) -> VEE
- C2 pad 2: VEE -> Net-(C2-Pad2)
- C3 pad 1: Net-(C3-Pad1) -> /VIN
- C4 pad 2: VEE -> GND
- C5 pad 1: Net-(C5-Pad1) -> /VIN
- C6 pad 2: VEE -> GND
- C7 pad 1: /SW+ -> VCC
- C7 pad 2: Net-(C7-Pad2) -> GND
- C8 pad 1: /SW- -> GND
- C8 pad 2: Net-(C8-Pad2) -> VEE
- L1 pad 1: /SW+ -> /VIN
- L1 pad 2: VCC -> Net-(L1-Pad2)
- L2 pad 1: /SW- -> /VIN
- L2 pad 2: GND -> Net-(D4-Pad2)
- R10 pad 1: VCC -> +15V
- R10 pad 2: Net-(C9-Pad2) -> Net-(R10-Pad2)
- R11 pad 1: GND -> Net-(R10-Pad2)
- R11 pad 2: Net-(C10-Pad2) -> GND
- R3 pad 2: VEE -> /VIN
- R4 pad 1: Net-(C3-Pad1) -> Net-(R4-Pad1)
- R4 pad 2: Net-(R2-Pad1) -> /VIN
- R5 pad 1: Net-(C4-Pad1) -> Net-(R5-Pad1)
- R5 pad 2: Net-(R3-Pad1) -> /VIN
- R6 pad 1: Net-(R6-Pad1) -> VCC
- R6 pad 2: GND -> Net-(C9-Pad2)
- R7 pad 1: Net-(R7-Pad1) -> Net-(C9-Pad2)
- R7 pad 2: VEE -> GND
- R8 pad 1: Net-(C9-Pad2) -> GND
- R8 pad 2: GND -> Net-(C10-Pad1)
- R9 pad 1: Net-(C10-Pad2) -> Net-(C10-Pad1)
- U1 pad 1: Net-(C7-Pad2) -> GND
- U1 pad 10: /VIN -> GND
- U1 pad 2: /SW+ -> /VIN
- U1 pad 3: Net-(C3-Pad1) -> Net-(R4-Pad1)
- U1 pad 4: Net-(R6-Pad1) -> Net-(C9-Pad2)
- U1 pad 5: Net-(R2-Pad1) -> Net-(R3-Pad1)
- U1 pad 6: Net-(C9-Pad2) -> Net-(R2-Pad1)
- U1 pad 7: Net-(C5-Pad1) -> Net-(C4-Pad1)
- U1 pad 8: (no net) -> GND
- U1 pad 9: /VIN -> GND
- U3 pad 7: VCC -> Net-(R10-Pad2)
- U4 pad 5: VEE -> Net-(R18-Pad2)
Routing:
- net -15V: track 2.76 -> 21.7 mm, vias 0 -> 8
- net +15V: track 1.77 -> 19.5 mm, vias 0 -> 8
- net Net-(C10-Pad1): track 0.00 -> 7.86 mm
- net GND: track 24.3 -> 18.2 mm, vias 34 -> 78
- net Net-(R5-Pad1): track 0.00 -> 5.83 mm
- net Net-(C3-Pad1): track 5.77 -> 0.00 mm
- net Net-(C2-Pad2): track 0.00 -> 5.69 mm, vias 0 -> 2
- net Net-(C9-Pad2): track 4.14 -> 9.57 mm
- net Net-(C10-Pad2): track 4.15 -> 0.00 mm
- net /VIN: track 23.8 -> 20.1 mm, vias 0 -> 16
- net /SW-: track 3.56 -> 0.00 mm
- net /SW+: track 3.54 -> 0.00 mm
- net VEE: track 17.9 -> 14.6 mm, vias 0 -> 28
- net Net-(C16-Pad2): track 3.05 -> 0.00 mm
- net Net-(C15-Pad1): track 3.05 -> 0.00 mm
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- added copper zone on B.Cu, net +15V
- added copper zone on B.Cu, net -15V
- added copper zone on B.Cu, net /VIN
- added copper zone on F.Cu, net Net-(C15-Pad1)
- added copper zone on F.Cu, net Net-(C16-Pad2)
- added copper zone on F.Cu, net Net-(D4-Pad2)
- added copper zone on F.Cu, net Net-(D5-Pad1)
- added copper zone on F.Cu, net Net-(L1-Pad2)
- removed copper zone on F.Cu, net /SW+
- removed copper zone on F.Cu, net /SW-
Other:
- net class Default: trace_width 0.25 -> 0.2; via_dia 0.8 -> 0.6; via_drill 0.4 -> 0.3
- net class Power: via_dia 0.8 -> 0.6; via_drill 0.4 -> 0.3
- rule via_min_size: 0.4 -> 0.6
- board text added: "2.0.0"
- board text removed: "1.0.0"
